File: PCB/PCB.kicad_pcb (KiCad board)
At the start: 2 copper layers, 3.6 x 3.2 mm, 279 parts, among them SW1 SW_Push, SW10 SW_Push, SW11 SW_Push, SW12 SW_Push, SW13 SW_Push, SW14 SW_Push, SW15 SW_Push, SW16 SW_Push, SW17 SW_Push, SW18 SW_Push, SW19 SW_Push, SW2 SW_Push, SW20 SW_Push, SW21 SW_Push, SW22 SW_Push, SW23 SW_Push, SW24 SW_Push, SW25 SW_Push, SW26 SW_Push, SW27 SW_Push, SW28 SW_Push, SW29 SW_Push, SW3 SW_Push, SW30 SW_Push, SW31 SW_Push, SW32 SW_Push, SW33 SW_Push, SW34 SW_Push, SW35 SW_Push, SW36 SW_Push, SW37 SW_Push, SW38 SW_Push, SW39 SW_Push, SW4 SW_Push, SW40 SW_Push, SW41 SW_Push, SW42 SW_Push, SW43 SW_Push, SW44 SW_Push, SW45 SW_Push, SW46 SW_Push, SW47 SW_Push, SW48 SW_Push, SW49 SW_Push, SW5 SW_Push, SW50 SW_Push, SW51 SW_Push, SW52 SW_Push, SW53 SW_Push, SW54 SW_Push, SW55 SW_Push, SW56 SW_Push, SW57 SW_Push, SW58 SW_Push, SW59 SW_Push, SW6 SW_Push, SW60 SW_Push, SW61 SW_Push, SW62 SW_Push, SW63 SW_Push, SW64 SW_Push, SW65 SW_Push, SW66 SW_Push, SW67 RotaryEncoder_Switch, SW7 SW_Push, SW8 SW_Push, SW9 SW_Push, U1 ER_OLEDM0.91_1x-I2C, U2 74AHCT125

Commit message: Update
Parts:
- added C64: 100nF, Capacitor_SMD:C_0805_2012Metric, F.Cu at (300.6, 116.3)
- added D131: SK6812MINI-E, LED_SMD:LED_SK6812MINI-E_3.2x2.8mm_P1.5mm_ReverseMount, F.Cu at (302.6, 112.3)
- turned D100 to 0 degrees
- turned D101 to 0 degrees
- turned D102 to 0 degrees
- turned D103 to 0 degrees
- turned D104 to 0 degrees
- turned D105 to 0 degrees
- turned D106 to 0 degrees
- turned D107 to 0 degrees
- turned D108 to 0 degrees
- turned D109 to 0 degrees
- turned D111 to 0 degrees
- turned D112 to 0 degrees
- turned D113 to 0 degrees
- turned D114 to 0 degrees
- turned D115 to 0 degrees
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Connections:
- D110 pad 4: unconnected-(D110-DOUT-Pad4) -> Net-(D110-DOUT)
- D111 pad 2: unconnected-(D111-DIN-Pad2) -> Net-(D110-DOUT)
- D123 pad 4: unconnected-(D123-DOUT-Pad4) -> Net-(D123-DOUT)
- D124 pad 2: unconnected-(D124-DIN-Pad2) -> Net-(D123-DOUT)
- D81 pad 4: unconnected-(D81-DOUT-Pad4) -> Net-(D81-DOUT)
- D82 pad 2: unconnected-(D82-DIN-Pad2) -> Net-(D81-DOUT)
- D96 pad 4: unconnected-(D96-DOUT-Pad4) -> Net-(D96-DOUT)
- D97 pad 2: unconnected-(D97-DIN-Pad2) -> Net-(D96-DOUT)
Routing:
- net Net-(D81-DOUT): track 0.00 -> 342.7 mm
- net Net-(D96-DOUT): track 0.00 -> 339.1 mm
- net Net-(D80-DOUT): track 0.00 -> 82.3 mm, vias 0 -> 2
- net Net-(D95-DOUT): track 0.00 -> 77.8 mm, vias 0 -> 2
- net Net-(D79-DOUT): track 0.00 -> 25.3 mm
- net Net-(D97-DOUT): track 0.00 -> 22.9 mm
- net Net-(D94-DOUT): track 0.00 -> 20.3 mm
- net Net-(D82-DOUT): track 0.00 -> 20.1 mm
- net Net-(D70-DOUT): track 0.00 -> 15.8 mm
- net Net-(D103-DOUT): track 0.00 -> 15.8 mm
- net Net-(D88-DOUT): track 0.00 -> 15.8 mm
- net Net-(D93-DOUT): track 0.00 -> 15.7 mm
- net Net-(D78-DOUT): track 0.00 -> 15.7 mm
- net Net-(D89-DOUT): track 0.00 -> 15.7 mm
- net Net-(D72-DOUT): track 0.00 -> 15.7 mm
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
Commit message: Update
Parts:
- removed the C64 at (300.6, 116.3)
- removed the C64 at (262.7, 101.8)
- removed the D130 at (294.6, 102.2)
- removed the D130 at (270.8, 102.2)
- added C64: 100nF, Capacitor_SMD:C_0805_2012Metric, B.Cu at (267.4, 102.2)
- added D130: SK6812MINI-E, LED_SMD:LED_SK6812MINI-E_3.2x2.8mm_P1.5mm_ReverseMount, B.Cu at (261.9, 101.5)
- added R1: 4.7kΩ, Resistor_SMD:R_0805_2012Metric, F.Cu at (347.8, 48.7)
- added R2: 4.7kΩ, Resistor_SMD:R_0805_2012Metric, F.Cu at (348.8, 39.2)
- added R3: 330Ω, Resistor_SMD:R_0805_2012Metric, F.Cu at (305.0, 17.8)
- D1, D10, D11, D12, D13, D131, D14, D15, D16, D17, D18, D19, D2, D20, D21, D22, D23, D24, D25, D26, D27, D28, D29, D3, D30, D31, D32, D33, D34, D35, D36, D37, D38, D39, D4, D40, D41, D42, D43, D44, D45, D46, D47, D48, D49, D5, D50, D51, D52, D53, D54, D55, D56, D57, D58, D59, D6, D60, D62, D63, D64, D65, D66, D7, D8, D9: moved to B.Cu
- SW1, SW10, SW11, SW12, SW13, SW14, SW15, SW17, SW18, SW19, SW2, SW20, SW21, SW22, SW23, SW24, SW25, SW26, SW27, SW28, SW3, SW30, SW32, SW33, SW34, SW35, SW36, SW37, SW38, SW39, SW4, SW40, SW41, SW42, SW43, SW44, SW45, SW46, SW47, SW48, SW49, SW5, SW50, SW51, SW52, SW53, SW54, SW55, SW56, SW57, SW6, SW61, SW66, SW7, SW8, SW9: footprint PCM_marbastlib-mx:SW_MX_1u -> PCM_marbastlib-mx:SW_MX_HS_CPG151101S11_1u
- SW16, SW29: footprint PCM_marbastlib-mx:SW_MX_1.5u -> PCM_marbastlib-mx:SW_MX_HS_CPG151101S11_1.5u
- SW31: footprint PCM_marbastlib-mx:SW_MX_1.75u -> PCM_marbastlib-mx:SW_MX_HS_CPG151101S11_1.75u
- SW58: footprint PCM_marbastlib-mx:SW_MX_1.25u -> PCM_marbastlib-mx:SW_MX_HS_CPG151101S11_1u
- SW59, SW60, SW62, SW63, SW64, SW65: footprint PCM_marbastlib-mx:SW_MX_1.25u -> PCM_marbastlib-mx:SW_MX_HS_CPG151101S11_1.25u
- moved H1 379.7 mm to (54.4, 181.1)
- moved H2 379.7 mm to (54.4, 189.0)
- moved H3 379.7 mm to (62.3, 181.1)
- moved H4 379.7 mm to (62.3, 189.0)
- moved H5 379.7 mm to (70.3, 181.1)
- moved H6 379.7 mm to (70.3, 189.0)
- moved D45 22.5 mm to (32.6, 86.8)
- moved D131 20.0 mm to (285.8, 101.5)
- moved C30 17.1 mm to (367.4, 45.1)
- moved D43 16.0 mm to (275.5, 67.8), turned to 180 degrees
- moved C44 15.2 mm to (367.4, 64.1)
- moved C15 14.3 mm to (367.4, 26.0)
- moved C57 14.3 mm to (367.4, 83.2)
- moved C66 14.3 mm to (367.4, 102.2)
- moved D15 11.3 mm to (361.2, 29.5), turned to 180 degrees
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Connections:
- C1 pad 1: VBUS -> GND
- C1 pad 2: Net-(D67-VDD) -> VBUS
- C10 pad 1: VBUS -> GND
- C10 pad 2: Net-(D76-VDD) -> VBUS
- C11 pad 1: VBUS -> GND
- C11 pad 2: Net-(D77-VDD) -> VBUS
- C12 pad 1: VBUS -> GND
- C12 pad 2: Net-(D78-VDD) -> VBUS
- C13 pad 1: VBUS -> GND
- C13 pad 2: Net-(D79-VDD) -> VBUS
- C14 pad 1: VBUS -> GND
- C14 pad 2: Net-(D80-VDD) -> VBUS
- C15 pad 1: VBUS -> GND
- C15 pad 2: Net-(D81-VDD) -> VBUS
- C16 pad 1: VBUS -> GND
- C16 pad 2: Net-(D82-VDD) -> VBUS
- C17 pad 1: VBUS -> GND
- C17 pad 2: Net-(D83-VDD) -> VBUS
- C18 pad 1: VBUS -> GND
- C18 pad 2: Net-(D84-VDD) -> VBUS
- C19 pad 1: VBUS -> GND
- C19 pad 2: Net-(D85-VDD) -> VBUS
- C2 pad 1: VBUS -> GND
- C2 pad 2: Net-(D68-VDD) -> VBUS
- C20 pad 1: VBUS -> GND
- C20 pad 2: Net-(D86-VDD) -> VBUS
- C21 pad 1: VBUS -> GND
- C21 pad 2: Net-(D87-VDD) -> VBUS
- C22 pad 1: VBUS -> GND
- C22 pad 2: Net-(D88-VDD) -> VBUS
- C23 pad 1: VBUS -> GND
- C23 pad 2: Net-(D89-VDD) -> VBUS
- C24 pad 1: VBUS -> GND
- C24 pad 2: Net-(D90-VDD) -> VBUS
- C25 pad 1: VBUS -> GND
- C25 pad 2: Net-(D91-VDD) -> VBUS
- C26 pad 1: VBUS -> GND
- C26 pad 2: Net-(D92-VDD) -> VBUS
- C27 pad 1: VBUS -> GND
- C27 pad 2: Net-(D93-VDD) -> VBUS
- C28 pad 1: VBUS -> GND
- C28 pad 2: Net-(D94-VDD) -> VBUS
- C29 pad 1: VBUS -> GND
- C29 pad 2: Net-(D95-VDD) -> VBUS
- C3 pad 1: VBUS -> GND
- C3 pad 2: Net-(D69-VDD) -> VBUS
- C30 pad 1: VBUS -> GND
- C30 pad 2: Net-(D96-VDD) -> VBUS
- C31 pad 1: VBUS -> GND
- C31 pad 2: Net-(D97-VDD) -> VBUS
- C32 pad 1: VBUS -> GND
- C32 pad 2: Net-(D98-VDD) -> VBUS
- C33 pad 1: VBUS -> GND
- C33 pad 2: Net-(D99-VDD) -> VBUS
- C34 pad 1: VBUS -> GND
- C34 pad 2: Net-(D100-VDD) -> VBUS
- C35 pad 1: VBUS -> GND
- C35 pad 2: Net-(D101-VDD) -> VBUS
- C36 pad 1: VBUS -> GND
- C36 pad 2: Net-(D102-VDD) -> VBUS
- C37 pad 1: VBUS -> GND
- C37 pad 2: Net-(D103-VDD) -> VBUS
- C38 pad 1: VBUS -> GND
- C38 pad 2: Net-(D104-VDD) -> VBUS
- C39 pad 1: VBUS -> GND
- C39 pad 2: Net-(D105-VDD) -> VBUS
- C4 pad 1: VBUS -> GND
- C4 pad 2: Net-(D70-VDD) -> VBUS
- C40 pad 1: VBUS -> GND
- C40 pad 2: Net-(D106-VDD) -> VBUS
- C41 pad 1: VBUS -> GND
- C41 pad 2: Net-(D107-VDD) -> VBUS
- C42 pad 1: VBUS -> GND
- C42 pad 2: Net-(D108-VDD) -> VBUS
- C43 pad 1: VBUS -> GND
- C43 pad 2: Net-(D109-VDD) -> VBUS
- C44 pad 1: VBUS -> GND
- C44 pad 2: Net-(D110-VDD) -> VBUS
- C45 pad 1: VBUS -> GND
- C45 pad 2: Net-(D111-VDD) -> VBUS
- C46 pad 1: VBUS -> GND
- C46 pad 2: Net-(D112-VDD) -> VBUS
- C47 pad 1: VBUS -> GND
- C47 pad 2: Net-(D113-VDD) -> VBUS
- C48 pad 1: VBUS -> GND
- C49 pad 1: VBUS -> GND
- C49 pad 2: Net-(D115-VDD) -> VBUS
- C5 pad 1: VBUS -> GND
- C5 pad 2: Net-(D71-VDD) -> VBUS
- C50 pad 1: VBUS -> GND
- C50 pad 2: Net-(D116-VDD) -> VBUS
- C51 pad 1: VBUS -> GND
- C51 pad 2: Net-(D117-VDD) -> VBUS
- C52 pad 1: VBUS -> GND
- C52 pad 2: Net-(D118-VDD) -> VBUS
- C53 pad 1: VBUS -> GND
- C53 pad 2: Net-(D119-VDD) -> VBUS
- C54 pad 1: VBUS -> GND
- C54 pad 2: Net-(D120-VDD) -> VBUS
- C55 pad 1: VBUS -> GND
- C55 pad 2: Net-(D121-VDD) -> VBUS
- C56 pad 1: VBUS -> GND
- C56 pad 2: Net-(D122-VDD) -> VBUS
- C57 pad 1: VBUS -> GND
- C57 pad 2: Net-(D123-VDD) -> VBUS
- C58 pad 1: VBUS -> GND
- C58 pad 2: Net-(D124-VDD) -> VBUS
- C59 pad 1: VBUS -> GND
- C59 pad 2: Net-(D125-VDD) -> VBUS
- C6 pad 1: VBUS -> GND
- C6 pad 2: Net-(D72-VDD) -> VBUS
- C60 pad 1: VBUS -> GND
- C60 pad 2: Net-(D126-VDD) -> VBUS
- C61 pad 1: VBUS -> GND
- C61 pad 2: Net-(D127-VDD) -> VBUS
- C62 pad 1: VBUS -> GND
- C62 pad 2: Net-(D128-VDD) -> VBUS
- C63 pad 1: VBUS -> GND
- C63 pad 2: Net-(D129-VDD) -> VBUS
- C65 pad 1: VBUS -> GND
- C65 pad 2: Net-(D131-VDD) -> VBUS
- C66 pad 1: VBUS -> GND
- C66 pad 2: Net-(D132-VDD) -> VBUS
- C7 pad 1: VBUS -> GND
- C7 pad 2: Net-(D73-VDD) -> VBUS
- C8 pad 1: VBUS -> GND
- C8 pad 2: Net-(D74-VDD) -> VBUS
- C9 pad 1: VBUS -> GND
- C9 pad 2: Net-(D75-VDD) -> VBUS
- D100 pad 3: Net-(D100-VDD) -> VBUS
- D101 pad 3: Net-(D101-VDD) -> VBUS
- D102 pad 3: Net-(D102-VDD) -> VBUS
- D103 pad 3: Net-(D103-VDD) -> VBUS
- D104 pad 3: Net-(D104-VDD) -> VBUS
- D105 pad 3: Net-(D105-VDD) -> VBUS
- D106 pad 3: Net-(D106-VDD) -> VBUS
- D107 pad 3: Net-(D107-VDD) -> VBUS
- D108 pad 3: Net-(D108-VDD) -> VBUS
- D109 pad 3: Net-(D109-VDD) -> VBUS
- D110 pad 3: Net-(D110-VDD) -> VBUS
- D111 pad 3: Net-(D111-VDD) -> VBUS
- D112 pad 3: Net-(D112-VDD) -> VBUS
- D113 pad 3: Net-(D113-VDD) -> VBUS
- D115 pad 3: Net-(D115-VDD) -> VBUS
- D116 pad 3: Net-(D116-VDD) -> VBUS
- D117 pad 3: Net-(D117-VDD) -> VBUS
- D118 pad 3: Net-(D118-VDD) -> VBUS
- D119 pad 3: Net-(D119-VDD) -> VBUS
- D120 pad 3: Net-(D120-VDD) -> VBUS
- D121 pad 3: Net-(D121-VDD) -> VBUS
- D122 pad 3: Net-(D122-VDD) -> VBUS
- D123 pad 3: Net-(D123-VDD) -> VBUS
- D124 pad 3: Net-(D124-VDD) -> VBUS
- D125 pad 3: Net-(D125-VDD) -> VBUS
- D126 pad 3: Net-(D126-VDD) -> VBUS
- D127 pad 3: Net-(D127-VDD) -> VBUS
- D128 pad 3: Net-(D128-VDD) -> VBUS
- D129 pad 3: Net-(D129-VDD) -> VBUS
- D131 pad 3: Net-(D131-VDD) -> VBUS
- D132 pad 3: Net-(D132-VDD) -> VBUS
- D67 pad 3: Net-(D67-VDD) -> VBUS
- D68 pad 3: Net-(D68-VDD) -> VBUS
- D69 pad 3: Net-(D69-VDD) -> VBUS
- D70 pad 3: Net-(D70-VDD) -> VBUS
- D71 pad 3: Net-(D71-VDD) -> VBUS
- D72 pad 3: Net-(D72-VDD) -> VBUS
- D73 pad 3: Net-(D73-VDD) -> VBUS
- D74 pad 3: Net-(D74-VDD) -> VBUS
- D75 pad 3: Net-(D75-VDD) -> VBUS
- D76 pad 3: Net-(D76-VDD) -> VBUS
- D77 pad 3: Net-(D77-VDD) -> VBUS
- D78 pad 3: Net-(D78-VDD) -> VBUS
- D79 pad 3: Net-(D79-VDD) -> VBUS
- D80 pad 3: Net-(D80-VDD) -> VBUS
- D81 pad 3: Net-(D81-VDD) -> VBUS
- D82 pad 3: Net-(D82-VDD) -> VBUS
- D83 pad 3: Net-(D83-VDD) -> VBUS
- D84 pad 3: Net-(D84-VDD) -> VBUS
- D85 pad 3: Net-(D85-VDD) -> VBUS
- D86 pad 3: Net-(D86-VDD) -> VBUS
- D87 pad 3: Net-(D87-VDD) -> VBUS
- D88 pad 3: Net-(D88-VDD) -> VBUS
- D89 pad 3: Net-(D89-VDD) -> VBUS
- D90 pad 3: Net-(D90-VDD) -> VBUS
- D91 pad 3: Net-(D91-VDD) -> VBUS
- D92 pad 3: Net-(D92-VDD) -> VBUS
- D93 pad 3: Net-(D93-VDD) -> VBUS
- D94 pad 3: Net-(D94-VDD) -> VBUS
- D95 pad 3: Net-(D95-VDD) -> VBUS
- D96 pad 3: Net-(D96-VDD) -> VBUS
- D97 pad 3: Net-(D97-VDD) -> VBUS
- D98 pad 3: Net-(D98-VDD) -> VBUS
- D99 pad 3: Net-(D99-VDD) -> VBUS
- U2 pad 14: (no net) -> +3V3
- U2 pad 3: DIN_5V -> Net-(R3-Pad1)
- U2 pad 7: (no net) -> GND
Routing:
- net Net-(D110-DOUT): track 0.00 -> 398.4 mm, vias 0 -> 2
- net Net-(D123-DOUT): track 0.00 -> 390.8 mm, vias 0 -> 2
- net +3V3: track 0.00 -> 139.2 mm, vias 0 -> 2
- net VBUS: track 0.00 -> 115.9 mm
- net Net-(D122-DOUT): track 0.00 -> 85.7 mm
- net Net-(D109-DOUT): track 0.00 -> 80.9 mm
- net Net-(D131-DOUT): track 0.00 -> 71.4 mm
- net Net-(D126-DOUT): track 0.00 -> 66.6 mm
- net Net-(D127-DOUT): track 0.00 -> 66.6 mm
- net Net-(D96-DOUT): track 339.1 -> 391.6 mm, vias 0 -> 2
- net Net-(D81-DOUT): track 342.7 -> 392.0 mm, vias 0 -> 2
- net DIN: track 42.2 -> 0.00 mm
- net Net-(D121-DOUT): track 0.00 -> 30.9 mm
- net Net-(D108-DOUT): track 0.00 -> 26.1 mm
- net Net-(D111-DOUT): track 0.00 -> 26.1 mm
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