File: PCB/PCB.kicad_pcb (KiCad board)
At the start: 2 copper layers, 3.6 x 3.2 mm, 282 parts, among them SW1 SW_Push, SW10 SW_Push, SW11 SW_Push, SW12 SW_Push, SW13 SW_Push, SW14 SW_Push, SW15 SW_Push, SW16 SW_Push, SW17 SW_Push, SW18 SW_Push, SW19 SW_Push, SW2 SW_Push, SW20 SW_Push, SW21 SW_Push, SW22 SW_Push, SW23 SW_Push, SW24 SW_Push, SW25 SW_Push, SW26 SW_Push, SW27 SW_Push, SW28 SW_Push, SW29 SW_Push, SW3 SW_Push, SW30 SW_Push, SW31 SW_Push, SW32 SW_Push, SW33 SW_Push, SW34 SW_Push, SW35 SW_Push, SW36 SW_Push, SW37 SW_Push, SW38 SW_Push, SW39 SW_Push, SW4 SW_Push, SW40 SW_Push, SW41 SW_Push, SW42 SW_Push, SW43 SW_Push, SW44 SW_Push, SW45 SW_Push, SW46 SW_Push, SW47 SW_Push, SW48 SW_Push, SW49 SW_Push, SW5 SW_Push, SW50 SW_Push, SW51 SW_Push, SW52 SW_Push, SW53 SW_Push, SW54 SW_Push, SW55 SW_Push, SW56 SW_Push, SW57 SW_Push, SW58 SW_Push, SW59 SW_Push, SW6 SW_Push, SW60 SW_Push, SW61 SW_Push, SW62 SW_Push, SW63 SW_Push, SW64 SW_Push, SW65 SW_Push, SW66 SW_Push, SW67 RotaryEncoder_Switch, SW7 SW_Push, SW8 SW_Push, SW9 SW_Push, U1 ER_OLEDM0.91_1x-I2C, U2 74AHCT125

Commit message: Update
Parts:
- added C67: 47µF, Capacitor_SMD:C_1206_3216Metric, F.Cu at (347.8, 14.2)
- added R4: 10kΩ, Resistor_SMD:R_0805_2012Metric, F.Cu at (346.4, 18.4)
Connections:
- A1 pad 37: unconnected-(A1-3V3_EN-Pad37) -> VSYS
- A1 pad 39: unconnected-(A1-VSYS-Pad39) -> VSYS
- C48 pad 2: Net-(D114-VDD) -> VBUS
- D114 pad 3: Net-(D114-VDD) -> VBUS
- D82 pad 1: unconnected-(D82-VSS-Pad1) -> GND
- U2 pad 14: +3V3 -> VBUS
Routing:
- net VBUS: track 115.9 -> 1027.8 mm, vias 0 -> 20
- net +3V3: track 139.2 -> 144.4 mm
- net VSYS: track 0.00 -> 4.76 mm
- net GND: track 0.00 -> 3.57 mm
- net Net-(D114-VDD): track 1.78 -> 0.00 mm

Commit message: Update
Routing:
- net VBUS: track 1027.8 -> 1918.3 mm, vias 20 -> 10
- net /ROW4: track 0.00 -> 347.7 mm
- net /ROW3: track 0.00 -> 343.0 mm, vias 0 -> 1
- net /COL14: track 0.00 -> 83.2 mm, vias 0 -> 6
- net Net-(D56-A): track 0.00 -> 43.9 mm, vias 0 -> 2
- net Net-(D46-A): track 0.00 -> 41.4 mm, vias 0 -> 2
- net +3V3: track 144.4 -> 113.4 mm
- net Net-(D60-A): track 0.00 -> 17.2 mm, vias 0 -> 1
- net Net-(D59-A): track 0.00 -> 17.1 mm, vias 0 -> 1
- net Net-(D61-A): track 0.00 -> 15.2 mm, vias 0 -> 1
- net Net-(D30-A): track 0.00 -> 15.1 mm, vias 0 -> 2
- net Net-(D57-A): track 0.00 -> 14.4 mm, vias 0 -> 1
- net Net-(D66-A): track 0.00 -> 14.3 mm, vias 0 -> 1
- net Net-(D15-A): track 0.00 -> 14.3 mm
- net Net-(D44-A): track 0.00 -> 14.3 mm
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
Commit message: Update
Routing:
- net /ROW2: track 0.00 -> 413.2 mm, vias 0 -> 6
- net /ROW1: track 0.00 -> 349.2 mm, vias 0 -> 1
- net /ROW0: track 0.00 -> 325.7 mm
- net /ROW4: track 347.7 -> 443.5 mm, vias 0 -> 7
- net /ROW3: track 343.0 -> 425.1 mm, vias 1 -> 9
- net /COL13: track 0.00 -> 34.8 mm, vias 0 -> 2
- net Net-(D46-A): track 41.4 -> 14.3 mm, vias 2 -> 0
- net /COL12: track 0.00 -> 24.3 mm, vias 0 -> 2
- net Net-(D12-A): track 0.00 -> 14.3 mm
- net Net-(D24-A): track 0.00 -> 14.3 mm
- net Net-(D43-A): track 0.00 -> 14.3 mm
- net Net-(D40-A): track 0.00 -> 14.3 mm
- net Net-(D7-A): track 0.00 -> 14.3 mm
- net Net-(D51-A): track 0.00 -> 14.3 mm
- net Net-(D5-A): track 0.00 -> 14.3 mm
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
Commit message: Update
Routing:
- net /COL0: track 0.00 -> 414.7 mm, vias 0 -> 10
- net /COL1: track 0.00 -> 408.1 mm, vias 0 -> 11
- net /COL2: track 0.00 -> 385.7 mm, vias 0 -> 11
- net /COL4: track 0.00 -> 361.4 mm, vias 0 -> 11
- net /ROW1: track 349.2 -> 709.4 mm, vias 1 -> 2
- net /COL3: track 0.00 -> 342.3 mm, vias 0 -> 9
- net /ROW4: track 443.5 -> 777.4 mm, vias 7 -> 1
- net /ROW3: track 425.1 -> 757.9 mm, vias 9 -> 2
- net /ROW2: track 413.2 -> 732.8 mm, vias 6 -> 3
- net /COL5: track 0.00 -> 312.3 mm, vias 0 -> 10
- net /COL6: track 0.00 -> 293.5 mm, vias 0 -> 11
- net /COL7: track 0.00 -> 282.6 mm, vias 0 -> 11
- net /COL8: track 0.00 -> 282.4 mm, vias 0 -> 13
- net /COL9: track 0.00 -> 275.5 mm, vias 0 -> 13
- net /COL11: track 0.00 -> 264.8 mm, vias 0 -> 11
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- added copper zone on B.Cu, net Net-(D109-DOUT)
- added copper zone on F.Cu, net Net-(D109-DOUT)
