File: PCB/PCB.kicad_sch (KiCad schematic)
At the start: 144 parts, among them SW1 SW_Push, SW10 SW_Push, SW11 SW_Push, SW12 SW_Push, SW13 SW_Push, SW14 SW_Push, SW15 SW_Push, SW16 SW_Push, SW17 SW_Push, SW18 SW_Push, SW19 SW_Push, SW2 SW_Push, SW20 SW_Push, SW21 SW_Push, SW22 SW_Push, SW23 SW_Push, SW24 SW_Push, SW25 SW_Push, SW26 SW_Push, SW27 SW_Push, SW28 SW_Push, SW29 SW_Push, SW3 SW_Push, SW30 SW_Push, SW31 SW_Push, SW32 SW_Push, SW33 SW_Push, SW34 SW_Push, SW35 SW_Push, SW36 SW_Push, SW37 SW_Push, SW38 SW_Push, SW39 SW_Push, SW4 SW_Push, SW40 SW_Push, SW41 SW_Push, SW42 SW_Push, SW43 SW_Push, SW44 SW_Push, SW45 SW_Push, SW46 SW_Push, SW47 SW_Push, SW48 SW_Push, SW49 SW_Push, SW5 SW_Push, SW50 SW_Push, SW51 SW_Push, SW52 SW_Push, SW53 SW_Push, SW54 SW_Push, SW55 SW_Push, SW56 SW_Push, SW57 SW_Push, SW58 SW_Push, SW59 SW_Push, SW6 SW_Push, SW60 SW_Push, SW61 SW_Push, SW62 SW_Push, SW63 SW_Push, SW64 SW_Push, SW65 SW_Push, SW66 SW_Push, SW7 SW_Push, SW8 SW_Push, SW9 SW_Push

Commit message: Update
Parts:
- added C10, C11, C12, C13, C14, C15, C16, C17, C18, C19, C2, C20, C21, C22, C23, C24, C25, C26, C27, C28, C29, C3, C30, C31, C32, C33, C34, C35, C36, C37, C38, C39, C4, C40, C42, C43, C44, C45, C46, C47, C48, C49, C5, C50, C51, C52, C53, C56, C57, C58, C59, C6, C60, C62, C66, C67, C68, C7, C70, C71, C8, C9: 100nF, symbol Device:C
- added D100, D101, D102, D103, D104, D105, D106, D107, D108, D109, D110, D111, D112, D113, D114, D115, D116, D117, D118, D119, D120, D121, D122, D123, D124, D125, D126, D127, D128, D67, D68, D69, D70, D71, D72, D73, D74, D75, D76, D77, D78, D79, D80, D81, D82, D83, D84, D85, D86, D87, D88, D89, D90, D91, D92, D93, D94, D95, D96, D97, D98, D99: SK6812MINI-E, LED_SMD:LED_SK6812MINI-E_3.2x2.8mm_P1.5mm_ReverseMount, symbol LED:SK6812MINI-E
- added SW67: RotaryEncoder_Switch, symbol Device:RotaryEncoder_Switch
- added U1: ER_OLEDM0.91_1x-I2C, Display:ER_OLEDM0.91_1x-I2C, symbol Display_Graphic:ER_OLEDM0.91_1x-I2C
- H1, H2, H3, H4, H5, H6: footprint MountingHole:MountingHole_2.2mm_M2 -> MountingHole:MountingHole_3.2mm_M3
Connections:
- net GND: now reaches A1.13 (GND), A1.18 (GND), A1.23 (GND), A1.28 (GND), A1.3 (GND), A1.38 (GND), A1.8 (GND)
- net GND: now also A1.33 (AGND), D100.1 (VSS), D101.1 (VSS), D102.1 (VSS), D103.1 (VSS), D104.1 (VSS), D105.1 (VSS), D106.1 (VSS), D107.1 (VSS), D108.1 (VSS), D109.1 (VSS), D110.1 (VSS), D111.1 (VSS), D112.1 (VSS), D113.1 (VSS), D114.1 (VSS), D115.1 (VSS), D116.1 (VSS), D117.1 (VSS), D118.1 (VSS), D119.1 (VSS), D120.1 (VSS), D121.1 (VSS), D122.1 (VSS), D123.1 (VSS), D124.1 (VSS), D125.1 (VSS), D126.1 (VSS), D127.1 (VSS), D128.1 (VSS), D67.1 (VSS), D68.1 (VSS), D69.1 (VSS), D70.1 (VSS), D71.1 (VSS), D72.1 (VSS), D73.1 (VSS), D74.1 (VSS), D75.1 (VSS), D76.1 (VSS), D77.1 (VSS), D78.1 (VSS), D79.1 (VSS), D80.1 (VSS), D82.1 (VSS), D83.1 (VSS), D84.1 (VSS), D85.1 (VSS), D86.1 (VSS), D87.1 (VSS), D88.1 (VSS), D89.1 (VSS), D90.1 (VSS), D91.1 (VSS), D92.1 (VSS), D93.1 (VSS), D94.1 (VSS), D95.1 (VSS), D96.1 (VSS), D97.1 (VSS), D98.1 (VSS), D99.1 (VSS), SW67.C, SW67.S1, U1.1 (GND)
- net at A1.26 (GPIO20): now also U1.4 (SDA)
- net at A1.27 (GPIO21): now also U1.3 (SCL)
- net DIN: now reaches A1.29 (GPIO22)
- net DIN: now also D67.2 (DIN)
- net at A1.31 (GPIO26_ADC0): now also SW67.A
- net at A1.32 (GPIO27_ADC1): now also SW67.B
- net at A1.34 (GPIO28_ADC2): now also SW67.S2
- net +3V3: now reaches A1.36 (3V3)
- net +3V3: now also U1.2 (VCC)
- net VBUS: now reaches A1.40 (VBUS)
- net VBUS: now also C10.1, C11.1, C12.1, C13.1, C14.1, C15.1, C16.1, C17.1, C18.1, C19.1, C2.1, C20.1, C21.1, C22.1, C23.1, C24.1, C25.1, C26.1, C27.1, C28.1, C29.1, C3.1, C30.1, C31.1, C32.1, C33.1, C34.1, C35.1, C36.1, C37.1, C38.1, C39.1, C4.1, C40.1, C42.1, C43.1, C44.1, C45.1, C46.1, C47.1, C48.1, C49.1, C5.1, C50.1, C51.1, C52.1, C53.1, C56.1, C57.1, C58.1, C59.1, C6.1, C60.1, C62.1, C66.1, C67.1, C68.1, C7.1, C70.1, C71.1, C8.1, C9.1
- new net: C48.2, D112.3 (VDD)
- new net: C6.2, D71.3 (VDD)
- new net: D86.4 (DOUT), D87.2 (DIN)
- new net: C22.2, D87.3 (VDD)
- new net: D87.4 (DOUT), D88.2 (DIN)
- new net: D88.4 (DOUT), D89.2 (DIN)
- new net: C24.2, D89.3 (VDD)
- new net: D89.4 (DOUT), D90.2 (DIN)
- new net: C9.2, D74.3 (VDD)
- new net: C21.2, D86.3 (VDD)
- new net: D74.4 (DOUT), D75.2 (DIN)
- new net: C10.2, D75.3 (VDD)
- new net: D75.4 (DOUT), D76.2 (DIN)
- new net: C46.2, D110.3 (VDD)
- new net: C68.2, D126.3 (VDD)
- new net: C27.2, D92.3 (VDD)
- new net: D81.4 (DOUT), D82.2 (DIN)
- new net: C17.2, D82.3 (VDD)
- new net: D82.4 (DOUT), D83.2 (DIN)
- new net: D100.4 (DOUT), D101.2 (DIN)
- new net: C36.2, D101.3 (VDD)
- new net: D101.4 (DOUT), D102.2 (DIN)
- new net: D95.4 (DOUT), D96.2 (DIN)
- new net: C31.2, D96.3 (VDD)
- new net: D96.4 (DOUT), D97.2 (DIN)
- new net: D68.4 (DOUT), D69.2 (DIN)
- new net: C4.2, D69.3 (VDD)
- new net: D69.4 (DOUT), D70.2 (DIN)
- new net: D79.4 (DOUT), D80.2 (DIN)
- new net: C15.2, D80.3 (VDD)
- new net: D91.4 (DOUT), D92.2 (DIN)
- new net: D92.4 (DOUT), D93.2 (DIN)
- new net: D97.4 (DOUT), D98.2 (DIN)
- new net: C33.2, D98.3 (VDD)
- new net: D98.4 (DOUT), D99.2 (DIN)
- new net: D117.4 (DOUT), D118.2 (DIN)
- new net: C56.2, D118.3 (VDD)
- new net: D118.4 (DOUT), D119.2 (DIN)
- new net: C57.2, D119.3 (VDD)
- new net: C26.2, D91.3 (VDD)
- new net: D113.4 (DOUT), D114.2 (DIN)
- new net: C50.2, D114.3 (VDD)
- new net: D114.4 (DOUT), D115.2 (DIN)
- new net: D83.4 (DOUT), D84.2 (DIN)
- new net: C19.2, D84.3 (VDD)
- new net: D84.4 (DOUT), D85.2 (DIN)
- new net: D105.4 (DOUT), D106.2 (DIN)
- new net: C42.2, D106.3 (VDD)
- new net: D106.4 (DOUT), D107.2 (DIN)
- new net: D126.4 (DOUT), D127.2 (DIN)
- new net: C70.2, D127.3 (VDD)
- new net: D127.4 (DOUT), D128.2 (DIN)
- new net: D108.4 (DOUT), D109.2 (DIN)
- new net: C45.2, D109.3 (VDD)
- new net: D109.4 (DOUT), D110.2 (DIN)
- new net: D110.4 (DOUT), D111.2 (DIN)
- new net: C14.2, D79.3 (VDD)
- new net: C62.2, D123.3 (VDD)
- new net: D104.4 (DOUT), D105.2 (DIN)
- new net: C40.2, D105.3 (VDD)
- new net: C28.2, D93.3 (VDD)
- new net: D93.4 (DOUT), D94.2 (DIN)
- new net: C52.2, D116.3 (VDD)
- new net: C25.2, D90.3 (VDD)
- new net: C20.2, D85.3 (VDD)
- new net: D85.4 (DOUT), D86.2 (DIN)
- new net: C59.2, D121.3 (VDD)
- new net: D67.4 (DOUT), D68.2 (DIN)
- new net: C3.2, D68.3 (VDD)
- new net: C30.2, D95.3 (VDD)
- new net: D124.4 (DOUT), D125.2 (DIN)
- new net: C67.2, D125.3 (VDD)
- new net: D125.4 (DOUT), D126.2 (DIN)
- new net: D73.4 (DOUT), D74.2 (DIN)
- new net: C16.2, D81.3 (VDD)
- new net: D72.4 (DOUT), D73.2 (DIN)
- new net: C8.2, D73.3 (VDD)
- new net: C18.2, D83.3 (VDD)
- new net: C51.2, D115.3 (VDD)
- new net: C2.2, D67.3 (VDD)
- new net: C47.2, D111.3 (VDD)
- new net: D76.4 (DOUT), D77.2 (DIN)
- new net: C12.2, D77.3 (VDD)
- new net: D77.4 (DOUT), D78.2 (DIN)
- new net: C11.2, D76.3 (VDD)
- new net: C43.2, D107.3 (VDD)
- new net: C58.2, D120.3 (VDD)
- new net: D120.4 (DOUT), D121.2 (DIN)
- new net: D90.4 (DOUT), D91.2 (DIN)
- new net: C44.2, D108.3 (VDD)
- new net: C37.2, D102.3 (VDD)
- new net: D102.4 (DOUT), D103.2 (DIN)
- new net: C53.2, D117.3 (VDD)
- new net: C38.2, D103.3 (VDD)
- new net: D103.4 (DOUT), D104.2 (DIN)
- new net: C29.2, D94.3 (VDD)
- new net: D78.4 (DOUT), D79.2 (DIN)
- new net: D100.2 (DIN), D99.4 (DOUT)
- new net: C35.2, D100.3 (VDD)
- new net: D122.4 (DOUT), D123.2 (DIN)
- new net: D123.4 (DOUT), D124.2 (DIN)
- new net: D111.4 (DOUT), D112.2 (DIN)
- new net: C49.2, D113.3 (VDD)
- new net: C34.2, D99.3 (VDD)
- new net: C39.2, D104.3 (VDD)
- new net: C13.2, D78.3 (VDD)
- new net: D121.4 (DOUT), D122.2 (DIN)
- new net: C71.2, D128.3 (VDD)
- new net: C60.2, D122.3 (VDD)
- new net: C32.2, D97.3 (VDD)
- new net: C23.2, D88.3 (VDD)
- new net: D116.4 (DOUT), D117.2 (DIN)
- new net: C7.2, D72.3 (VDD)
- new net: C66.2, D124.3 (VDD)
- new net: D112.4 (DOUT), D113.2 (DIN)
- new net: D71.4 (DOUT), D72.2 (DIN)
- new net: D115.4 (DOUT), D116.2 (DIN)
- new net: D70.4 (DOUT), D71.2 (DIN)
- new net: C5.2, D70.3 (VDD)
- no-connect marks 0 -> 2
Other:
- moved on the sheet: A1, H5, H6

Commit message: Update
Parts:
- removed C68: 100nF, symbol Device:C
- removed D126: SK6812MINI-E, LED_SMD:LED_SK6812MINI-E_3.2x2.8mm_P1.5mm_ReverseMount, symbol LED:SK6812MINI-E
- added C15, C30, C44, C57, C66: 100nF, Capacitor_SMD:C_0805_2012Metric, symbol Device:C
- added D110, D123, D132, D81, D96: SK6812MINI-E, LED_SMD:LED_SK6812MINI-E_3.2x2.8mm_P1.5mm_ReverseMount, symbol LED:SK6812MINI-E
- added U2: 74AHCT125, Package_SO:SOIC-14_3.9x8.7mm_P1.27mm, symbol 74xx:74AHCT125
- C1: renamed from C2; footprint (none) -> Capacitor_SMD:C_0805_2012Metric
- C10: renamed from C11; footprint (none) -> Capacitor_SMD:C_0805_2012Metric
- C11: renamed from C12; footprint (none) -> Capacitor_SMD:C_0805_2012Metric
- C12: renamed from C13; footprint (none) -> Capacitor_SMD:C_0805_2012Metric
- C13: renamed from C14; footprint (none) -> Capacitor_SMD:C_0805_2012Metric
- C14: renamed from C15; footprint (none) -> Capacitor_SMD:C_0805_2012Metric
- C16, C17, C18, C19, C20, C21, C22, C23, C24, C25, C26, C27, C28, C29, C42, C43, C58, C59, C60: footprint (none) -> Capacitor_SMD:C_0805_2012Metric
- C2: renamed from C3; footprint (none) -> Capacitor_SMD:C_0805_2012Metric
- C3: renamed from C4; footprint (none) -> Capacitor_SMD:C_0805_2012Metric
- C31: renamed from C30; footprint (none) -> Capacitor_SMD:C_0805_2012Metric
- C32: renamed from C31; footprint (none) -> Capacitor_SMD:C_0805_2012Metric
- C33: renamed from C32; footprint (none) -> Capacitor_SMD:C_0805_2012Metric
- C34: renamed from C33; footprint (none) -> Capacitor_SMD:C_0805_2012Metric
- C35: renamed from C34; footprint (none) -> Capacitor_SMD:C_0805_2012Metric
- C36: renamed from C35; footprint (none) -> Capacitor_SMD:C_0805_2012Metric
- C37: renamed from C36; footprint (none) -> Capacitor_SMD:C_0805_2012Metric
- C38: renamed from C37; footprint (none) -> Capacitor_SMD:C_0805_2012Metric
- C39: renamed from C38; footprint (none) -> Capacitor_SMD:C_0805_2012Metric
- C4: renamed from C5; footprint (none) -> Capacitor_SMD:C_0805_2012Metric
- C40: renamed from C39; footprint (none) -> Capacitor_SMD:C_0805_2012Metric
- C41: renamed from C40; footprint (none) -> Capacitor_SMD:C_0805_2012Metric
- C45: renamed from C44; footprint (none) -> Capacitor_SMD:C_0805_2012Metric
- C46: renamed from C45; footprint (none) -> Capacitor_SMD:C_0805_2012Metric
- C47: renamed from C46; footprint (none) -> Capacitor_SMD:C_0805_2012Metric
- C48: renamed from C47; footprint (none) -> Capacitor_SMD:C_0805_2012Metric
- C49: renamed from C48; footprint (none) -> Capacitor_SMD:C_0805_2012Metric
- C5: renamed from C6; footprint (none) -> Capacitor_SMD:C_0805_2012Metric
- C50: renamed from C49; footprint (none) -> Capacitor_SMD:C_0805_2012Metric
- C51: renamed from C50; footprint (none) -> Capacitor_SMD:C_0805_2012Metric
- C52: renamed from C51; footprint (none) -> Capacitor_SMD:C_0805_2012Metric
- C53: renamed from C52; footprint (none) -> Capacitor_SMD:C_0805_2012Metric
- C54: renamed from C53; footprint (none) -> Capacitor_SMD:C_0805_2012Metric
- C55: renamed from C56; footprint (none) -> Capacitor_SMD:C_0805_2012Metric
- C56: renamed from C57; footprint (none) -> Capacitor_SMD:C_0805_2012Metric
- C6: renamed from C7; footprint (none) -> Capacitor_SMD:C_0805_2012Metric
- C61: renamed from C62; footprint (none) -> Capacitor_SMD:C_0805_2012Metric
- C62: renamed from C66; footprint (none) -> Capacitor_SMD:C_0805_2012Metric
- C63: renamed from C67; footprint (none) -> Capacitor_SMD:C_0805_2012Metric
- C64: renamed from C70; footprint (none) -> Capacitor_SMD:C_0805_2012Metric
- C65: renamed from C71; footprint (none) -> Capacitor_SMD:C_0805_2012Metric
- C7: renamed from C8; footprint (none) -> Capacitor_SMD:C_0805_2012Metric
- C8: renamed from C9; footprint (none) -> Capacitor_SMD:C_0805_2012Metric
- C9: renamed from C10; footprint (none) -> Capacitor_SMD:C_0805_2012Metric
- SW29: footprint PCM_marbastlib-mx:SW_MX_1u -> PCM_marbastlib-mx:SW_MX_1.5u
- SW67: footprint (none) -> Rotary_Encoder:RotaryEncoder_Alps_EC11E-Switch_Vertical_H20mm
- renumbered D98 to D100, D99 to D101, D100 to D102, D101 to D103, D102 to D104, D103 to D105, D104 to D106, D105 to D107, D106 to D108, D107 to D109, D108 to D111, D109 to D112, D110 to D113, D111 to D114, D112 to D115, D113 to D116, D114 to D117, D115 to D118, D116 to D119, D117 to D120, D118 to D121, D119 to D122, D120 to D124, D121 to D125, D122 to D126, D123 to D127, D124 to D128, D125 to D129, D127 to D130, D128 to D131, D81 to D82, D82 to D83, D83 to D84, D84 to D85, D85 to D86, D86 to D87, D87 to D88, D88 to D89, D89 to D90, D90 to D91, D91 to D92, D92 to D93, D93 to D94, D94 to D95, D95 to D97, D96 to D98, D97 to D99
Connections:
- net DIN: now also U2.2; no longer D67.2 (DIN)
- net GND: now also D110.1 (VSS), D123.1 (VSS), D132.1 (VSS), D81.1 (VSS), D96.1 (VSS), U2.1
- net VBUS: now also C15.1, C30.1, C44.1, C57.1, C66.1
- net at D80.4 (DOUT): now also D81.2 (DIN)
- net at D122.4 (DOUT): now also D123.2 (DIN)
- net at D130.2 (DIN): now also D129.4 (DOUT)
- net at D109.4 (DOUT): now also D110.2 (DIN)
- net at D131.4 (DOUT): now also D132.2 (DIN)
- net at D95.4 (DOUT): now also D96.2 (DIN)
- new net: C57.2, D123.3 (VDD)
- new net: C66.2, D132.3 (VDD)
- new net: C30.2, D96.3 (VDD)
- new net: C44.2, D110.3 (VDD)
- new net: C15.2, D81.3 (VDD)
- new net DIN_5V: D67.2 (DIN), U2.3
Other:
- moved on the sheet: C1, C10, C11, C12, C13, C14, C16, C17, C18, C19, C2, C20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

Commit message: Update
Connections:
- net at D123.4 (DOUT): now also D124.2 (DIN)
- net at D110.4 (DOUT): now also D111.2 (DIN)
- net at D82.2 (DIN): now also D81.4 (DOUT)
- net at D97.2 (DIN): now also D96.4 (DOUT)
Changed lines of the file:
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@@
+	(wire
+		(pts
+			(xy 256.54 180.34) (xy 20.32 180.34)
+		)
+		(stroke
+			(width 0)
+			(type default)
+		)
+	)
+	(wire
+		(pts
+			(xy 256.54 222.25) (xy 21.59 222.25)
+		)
+		(stroke
+			(width 0)
+			(type default)
+		)
+	)
 	(wire
 		(pts
@@
 	(wire
 		(pts
+			(xy 256.54 201.93) (xy 21.59 201.93)
+		)
+		(stroke
+			(width 0)
+			(type default)
+		)
+	)
+	(wire
+		(pts
 			(xy 38.1 50.8) (xy 38.1 63.5)
 		)
@@
 	(wire
 		(pts
+			(xy 20.32 180.34) (xy 20.32 191.77)
+		)
+		(stroke
+			(width 0)
+			(type default)
+		)
+	)
+	(wire
+		(pts
 			(xy 50.8 76.2) (xy 50.8 88.9)
 		)
@@
 	(wire
 		(pts
+			(xy 21.59 233.68) (xy 27.94 233.68)
+		)
+		(stroke
+			(width 0)
+			(type default)
+		)
+	)
+	(wire
+		(pts
 			(xy 74.93 162.56) (xy 81.28 162.56)
 		)
@@
 	(wire
 		(pts
+			(xy 256.54 213.36) (xy 256.54 222.25)
+		)
+		(stroke
+			(width 0)
+			(type default)
+		)
+	)
+	(wire
+		(pts
 			(xy 114.3 50.8) (xy 114.3 63.5)
 		)
@@
 	(wire
 		(pts
+			(xy 21.59 213.36) (xy 27.94 213.36)
+		)
+		(stroke
+			(width 0)
+			(type default)
+		)
+	)
+	(wire
+		(pts
 			(xy 104.14 162.56) (xy 111.76 162.56)
 		)
@@
 	(wire
 		(pts
+			(xy 21.59 222.25) (xy 21.59 233.68)
+		)
+		(stroke
+			(width 0)
+			(type default)
+		)
+	)
+	(wire
+		(pts
 			(xy 111.76 45.72) (xy 124.46 45.72)
 		)
@@
 	(wire
 		(pts
+			(xy 16.51 170.18) (xy 27.94 170.18)
+		)
+		(stroke
+			(width 0)
+			(type default)
+		)
+	)
+	(wire
+		(pts
 			(xy 88.9 205.74) (xy 96.52 205.74)
 		)
@@
 	(wire
 		(pts
+			(xy 21.59 201.93) (xy 21.59 213.36)
+		)
+		(stroke
+			(width 0)
+			(type default)
+		)
+	)
+	(wire
+		(pts
 			(xy 149.86 205.74) (xy 157.48 205.74)
 		)
@@
 	(wire
 		(pts
+			(xy 256.54 191.77) (xy 256.54 201.93)
+		)
+		(stroke
+			(width 0)
+			(type default)
+		)
+	)
+	(wire
+		(pts
 			(xy 287.02 99.06) (xy 287.02 77.47)
 		)
@@
 	(wire
 		(pts
+			(xy 256.54 127) (xy 16.51 127)
+		)
+		(stroke
+			(width 0)
+			(type default)
+		)
+	)
+	(wire
+		(pts
 			(xy 309.88 93.98) (xy 309.88 99.06)
 		)
@@
 	(wire
 		(pts
+			(xy 256.54 151.13) (xy 256.54 127)
+		)
+		(stroke
+			(width 0)
+			(type default)
+		)
+	)
+	(wire
+		(pts
 			(xy 139.7 50.8) (xy 139.7 63.5)
 		)
@@
 	(wire
 		(pts
+			(xy 256.54 170.18) (xy 256.54 180.34)
+		)
+		(stroke
+			(width 0)
+			(type default)
+		)
+	)
+	(wire
+		(pts
 			(xy 111.76 71.12) (xy 124.46 71.12)
 		)
@@
 	(wire
 		(pts
+			(xy 20.32 191.77) (xy 27.94 191.77)
+		)
+		(stroke
+			(width 0)
+			(type default)
+		)
+	)
+	(wire
+		(pts
 			(xy 218.44 135.89) (xy 218.44 137.16)
 		)
 		(stroke
+			(width 0)
+			(type default)
+		)
+	)
+	(wire
+		(pts
+			(xy 16.51 127) (xy 16.51 170.18)
+		)
+		(stroke

Commit message: Update
Parts:
- added R1, R2: 4.7kΩ, Resistor_SMD:R_0805_2012Metric, symbol Device:R
- added R3: 330Ω, Resistor_SMD:R_0805_2012Metric, symbol Device:R
- added unit 5 of U2
- SW1, SW10, SW11, SW12, SW13, SW14, SW15, SW17, SW18, SW19, SW2, SW20, SW21, SW22, SW23, SW24, SW25, SW26, SW27, SW28, SW3, SW30, SW32, SW33, SW34, SW35, SW36, SW37, SW38, SW39, SW4, SW40, SW41, SW42, SW43, SW44, SW45, SW46, SW47, SW48, SW49, SW5, SW50, SW51, SW52, SW53, SW54, SW55, SW56, SW57, SW6, SW61, SW66, SW7, SW8, SW9: footprint PCM_marbastlib-mx:SW_MX_1u -> PCM_marbastlib-mx:SW_MX_HS_CPG151101S11_1u
- SW16, SW29: footprint PCM_marbastlib-mx:SW_MX_1.5u -> PCM_marbastlib-mx:SW_MX_HS_CPG151101S11_1.5u
- SW31: footprint PCM_marbastlib-mx:SW_MX_1.75u -> PCM_marbastlib-mx:SW_MX_HS_CPG151101S11_1.75u
- SW58: footprint PCM_marbastlib-mx:SW_MX_1.25u -> PCM_marbastlib-mx:SW_MX_HS_CPG151101S11_1u
- SW59, SW60, SW62, SW63, SW64, SW65: footprint PCM_marbastlib-mx:SW_MX_1.25u -> PCM_marbastlib-mx:SW_MX_HS_CPG151101S11_1.25u
Connections:
- net +3V3: now also R1.2, R2.2, U2.14 (VCC)
- net DIN_5V: now also R3.2; no longer U2.3
- net GND: now also C1.1, C10.1, C11.1, C12.1, C13.1, C14.1, C15.1, C16.1, C17.1, C18.1, C19.1, C2.1, C20.1, C21.1, C22.1, C23.1, C24.1, C25.1, C26.1, C27.1, C28.1, C29.1, C3.1, C30.1, C31.1, C32.1, C33.1, C34.1, C35.1, C36.1, C37.1, C38.1, C39.1, C4.1, C40.1, C41.1, C42.1, C43.1, C44.1, C45.1, C46.1, C47.1, C48.1, C49.1, C5.1, C50.1, C51.1, C52.1, C53.1, C54.1, C55.1, C56.1, C57.1, C58.1, C59.1, C6.1, C60.1, C61.1, C62.1, C63.1, C64.1, C65.1, C66.1, C7.1, C8.1, C9.1, U2.7 (GND)
- net VBUS: now also C1.2, C10.2, C11.2, C12.2, C13.2, C14.2, C15.2, C16.2, C17.2, C18.2, C19.2, C2.2, C20.2, C21.2, C22.2, C23.2, C24.2, C25.2, C26.2, C27.2, C28.2, C29.2, C3.2, C30.2, C31.2, C32.2, C33.2, C34.2, C35.2, C36.2, C37.2, C38.2, C39.2, C4.2, C40.2, C41.2, C42.2, C43.2, C44.2, C45.2, C46.2, C47.2, C49.2, C5.2, C50.2, C51.2, C52.2, C53.2, C54.2, C55.2, C56.2, C57.2, C58.2, C59.2, C6.2, C60.2, C61.2, C62.2, C63.2, C64.2, C65.2, C66.2, C7.2, C8.2, C9.2, D100.3 (VDD), D101.3 (VDD), D102.3 (VDD), D103.3 (VDD), D104.3 (VDD), D105.3 (VDD), D106.3 (VDD), D107.3 (VDD), D108.3 (VDD), D109.3 (VDD), D110.3 (VDD), D111.3 (VDD), D112.3 (VDD), D113.3 (VDD), D115.3 (VDD), D116.3 (VDD), D117.3 (VDD), D118.3 (VDD), D119.3 (VDD), D120.3 (VDD), D121.3 (VDD), D122.3 (VDD), D123.3 (VDD), D124.3 (VDD), D125.3 (VDD), D126.3 (VDD), D127.3 (VDD), D128.3 (VDD), D129.3 (VDD), D130.3 (VDD), D131.3 (VDD), D132.3 (VDD), D67.3 (VDD), D68.3 (VDD), D69.3 (VDD), D70.3 (VDD), D71.3 (VDD), D72.3 (VDD), D73.3 (VDD), D74.3 (VDD), D75.3 (VDD), D76.3 (VDD), D77.3 (VDD), D78.3 (VDD), D79.3 (VDD), D80.3 (VDD), D81.3 (VDD), D82.3 (VDD), D83.3 (VDD), D84.3 (VDD), D85.3 (VDD), D86.3 (VDD), D87.3 (VDD), D88.3 (VDD), D89.3 (VDD), D90.3 (VDD), D91.3 (VDD), D92.3 (VDD), D93.3 (VDD), D94.3 (VDD), D95.3 (VDD), D96.3 (VDD), D97.3 (VDD), D98.3 (VDD), D99.3 (VDD); no longer C1.1, C10.1, C11.1, C12.1, C13.1, C14.1, C15.1, C16.1, C17.1, C18.1, C19.1, C2.1, C20.1, C21.1, C22.1, C23.1, C24.1, C25.1, C26.1, C27.1, C28.1, C29.1, C3.1, C30.1, C31.1, C32.1, C33.1, C34.1, C35.1, C36.1, C37.1, C38.1, C39.1, C4.1, C40.1, C41.1, C42.1, C43.1, C44.1, C45.1, C46.1, C47.1, C48.1, C49.1, C5.1, C50.1, C51.1, C52.1, C53.1, C54.1, C55.1, C56.1, C57.1, C58.1, C59.1, C6.1, C60.1, C61.1, C62.1, C63.1, C64.1, C65.1, C66.1, C7.1, C8.1, C9.1
- net at A1.27 (GPIO21), U1.3 (SCL): now also R2.1
- net at A1.26 (GPIO20), U1.4 (SDA): now also R1.1
- new net: R3.1, U2.3

Commit message: Update
Parts:
- added C67: 47µF, Capacitor_SMD:C_1206_3216Metric, symbol Device:C
Connections:
- net +3V3: no longer U2.14 (VCC)
- net GND: now also D82.1 (VSS)
- net VBUS: now also C48.2, D114.3 (VDD), U2.14 (VCC), C67.1
- net VSYS: now reaches A1.37 (3V3_EN)
- net VSYS: now also A1.39 (VSYS), C67.2
- no-connect marks 2 -> 3
